Commit message: add colors

File: src/my_robot/urdf/my_robot.xacro (robot description, xacro)
@@ -101,5 +101,5 @@
       </geometry>
     </collision>
-    <visual name='visual'>
+    <visual>
       <origin xyz='0 0 0' rpy='0 1.5707 1.5707' />
       <geometry>
@@ -125,5 +125,5 @@
       </geometry>
     </collision>
-    <visual name='visual'>
+    <visual>
       <origin xyz='0 0 0' rpy='0 1.5707 1.5707' />
       <geometry>
@@ -149,5 +149,5 @@
       </geometry>
     </collision>
-    <visual name='visual'>
+    <visual>
       <origin xyz='0 0 0' rpy='0 0 0' />
       <geometry>
@@ -180,6 +180,21 @@
     </visual>
   </link>
-  <gazebo reference='left_wheel'>
+  <gazebo reference="left_wheel">
     <material>Gazebo/Green</material>
   </gazebo>
+  <gazebo reference="right_wheel">
+    <material>Gazebo/Green</material>
+  </gazebo>
+  <gazebo reference="chassis">
+    <material>Gazebo/Orange</material>
+  </gazebo>
+  <gazebo reference="chassis_back_caster_visual">
+    <material>Gazebo/Black</material>
+  </gazebo>
+  <gazebo reference="chassis_front_caster_visual">
+    <material>Gazebo/Black</material>
+  </gazebo>
+  <gazebo reference="camera">
+    <material>Gazebo/Red</material>
+  </gazebo>
 </robot>

Commit message: add mapping

File: src/my_robot/urdf/my_robot.xacro (robot description, xacro)
@@ -36,4 +36,11 @@
     <axis xyz='0 1 0' rpy='0 0 0' />
   </joint>
+  <joint name='camera_optical_joint' type='fixed'>
+     <origin xyz='0 0 0' rpy='-1.5707 0 -1.5707' />
+     <parent link='camera' />
+     <child link='camera_link_optical' />
+  </joint>
+  <link name='camera_link_optical'>
+  </link>
   <link name='chassis'>
     <pose>0 0 0.1 0 0 0</pose>
